Commit message: fix

File: urdf/camina.urdf (robot description, URDF)
Before this commit: robot cibo, 7 links, 6 joints
Links:
- removed link camera_01_link
- removed link camera_02_link
- removed link horizontal_bar_link
- removed link map
- removed link pedestal_link
- removed link vertical_bar_link
- added link camera_front_depth_frame; visual box size=0.0123 0.0653 0.0225
- added link camera_link
- added link camera_rear_depth_frame; visual box size=0.0123 0.0653 0.0225
Joints:
- removed joint base_pedestal_joint
- removed joint camera_01_joint
- removed joint camera_02_joint
- removed joint pedestal_vertical_joint
- removed joint vertical_horizontal_joint
- added joint camera_front_joint: type fixed, parent camera_link, child camera_front_depth_frame, origin xyz=0.0 0.0 1.0 rpy=0 0 0
- added joint camera_rear_joint: type fixed, parent camera_link, child camera_rear_depth_frame, origin xyz=4.0 0.0 1.0 rpy=0 0 3.14
- joint map_base_joint: child base_link -> camera_link; parent map -> base_link

Commit message: fix

File: urdf/camina.urdf (robot description, URDF)
Before this commit: robot cibo, 3 links, 2 joints
Links:
- added link camera_rear_depth_optical_frame
- added link camera_rear_link; visual box size=0.0123 0.0653 0.0225
Joints:
- added joint camera_rear_joint: type fixed, parent base_link, child camera_rear_link, origin xyz=3.0 0.0 1.0 rpy=0 0 3.14
- added joint camera_rear_optical_joint: type fixed, parent camera_rear_link, child camera_rear_depth_optical_frame, origin xyz=0.0 0.0 0.0 rpy=-1.570796 0 -1.570796

Commit message: fix

File: urdf/camina.urdf (robot description, URDF)
Before this commit: robot cibo, 5 links, 4 joints
Joints:
- joint camera_front_joint: origin xyz=0.0 0.0 1.0 rpy=0 0 0 -> xyz=0.0 0.0 0.9 rpy=0 0 0
- joint camera_rear_joint: origin xyz=3.0 0.0 1.0 rpy=0 0 3.14 -> xyz=3.8 0.0 0.9 rpy=0 0 3.14

Commit message: add: define materials for camera and lidar, and add lidar link and joint

File: urdf/camina.urdf (robot description, URDF)
Before this commit: robot cibo, 5 links, 4 joints
Links:
- added link laser; visual cylinder length=0.06 radius=0.1
Joints:
- added joint lidar_joint: type fixed, parent base_link, child laser, origin xyz=0.1 0 0.4 rpy=0 0 0

Commit message: fix

File: urdf/camina.urdf (robot description, URDF)
Before this commit: robot cibo, 6 links, 5 joints
Links:
- link laser: geometry visual cylinder length=0.1 radius=0.05

Commit message: fix

File: urdf/camina.urdf (robot description, URDF)
Before this commit: robot cibo, 6 links, 5 joints
Links:
- link camera_front_link: geometry visual box size=0.05 0.1 0.03
- link camera_rear_link: geometry visual box size=0.05 0.1 0.03

Commit message: fix

File: urdf/camina.urdf (robot description, URDF)
Before this commit: robot cibo, 6 links, 5 joints
Links:
- added link camera_front_depth_frame
Joints:
- added joint camera_front_depth_joint: type fixed, parent camera_front_link, child camera_front_depth_frame, origin xyz=0.0 0.0 0.0 rpy=0 0 0
- joint camera_front_optical_joint: parent camera_front_link -> camera_front_depth_frame

Commit message: fix

File: urdf/camina.urdf (robot description, URDF)
Before this commit: robot cibo, 7 links, 6 joints
Links:
- added link camera_front_color_frame
- added link camera_front_color_optical_frame
Joints:
- removed joint camera_front_optical_joint
- added joint camera_front_color_joint: type fixed, parent camera_front_link, child camera_front_color_frame, origin xyz=0.0 0.0 0.0 rpy=0 0 0
- added joint camera_front_color_optical_joint: type fixed, parent camera_front_color_frame, child camera_front_color_optical_frame, origin xyz=0.0 0.0 0.0 rpy=-1.570796 0 -1.570796
- added joint camera_front_depth_optical_joint: type fixed, parent camera_front_depth_frame, child camera_front_depth_optical_frame, origin xyz=0.0 0.0 0.0 rpy=-1.570796 0 -1.570796

Commit message: fix

File: urdf/camina.urdf (robot description, URDF)
Before this commit: robot cibo, 9 links, 8 joints
Links:
- added link camera_rear_color_frame
- added link camera_rear_color_optical_frame
Joints:
- added joint camera_rear_color_joint: type fixed, parent camera_rear_link, child camera_rear_color_frame, origin xyz=0.0 0.0 0.0 rpy=0 0 0
- added joint camera_rear_color_optical_joint: type fixed, parent camera_rear_color_frame, child camera_rear_color_optical_frame, origin xyz=0.0 0.0 0.0 rpy=-1.570796 0 -1.570796

Commit message: fix

File: urdf/camina.urdf (robot description, URDF)
Before this commit: robot cibo, 11 links, 10 joints
Links:
- added link camera_rear_depth_frame
Joints:
- removed joint camera_rear_optical_joint
- added joint camera_rear_depth_joint: type fixed, parent camera_rear_link, child camera_rear_depth_frame, origin xyz=0.0 0.0 0.0 rpy=0 0 0
- added joint camera_rear_depth_optical_joint: type fixed, parent camera_rear_depth_frame, child camera_rear_depth_optical_frame, origin xyz=0.0 0.0 0.0 rpy=-1.570796 0 -1.570796

Commit message: add base frame and joint for map and base_link

File: urdf/camina.urdf (robot description, URDF)
Before this commit: robot cibo, 12 links, 11 joints
Links:
- added link map
Joints:
- added joint base_map_joint: type fixed, parent map, child base_link

Commit message: fix

File: urdf/camina.urdf (robot description, URDF)
Before this commit: robot cibo, 13 links, 12 joints
Joints:
- joint camera_rear_joint: origin xyz=3.8 0.0 0.9 rpy=0 0 3.14 -> xyz=6.4 0.0 0.8 rpy=0 0 3.14
- joint lidar_joint: origin xyz=0.1 0 0.4 rpy=0 0 0 -> xyz=0.05 0 0.4 rpy=0 0 0
