Commit message: chore

File: urdf/camina.urdf (robot description, URDF)
Before this commit: robot cibo, 13 links, 12 joints
Joints:
- joint camera_rear_joint: origin xyz=6.4 0.0 0.8 rpy=0 0 3.14 -> xyz=5.0 0.0 0.8 rpy=0 0 3.14
- joint lidar_joint: origin xyz=0.05 0 0.4 rpy=0 0 0 -> xyz=0.00 0 0.4 rpy=0 0 0
